File: ReFlow PCB.kicad_pcb (KiCad board)
At the start: 2 copper layers, 78.2 x 78.5 mm, 23 parts, among them J1 Barrel_Jack_MountingPin, J2 Display OLED, J3 Conn_02x03_M, Q1 IRF3205N, SW1 SW_MEC_5E, SW2 SW_MEC_5E, SW3 SW_MEC_5E, U2 L7805, U3 ATtiny85-20S

Commit message: Add files via upload
Other:
- board text added: "70x50mm"
- board text removed: "70x50mm TinyReflow V1,2 CERN-OHL-P v2"
Changed lines of the file:
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@@
 		(layer "Edge.Cuts")
 	)
-	(gr_text "70x50mm TinyReflow V1,2 CERN-OHL-P v2"
+	(gr_text "70x50mm"
 		(at 108.5 119.5 270)
 		(layer "F.SilkS")
@@
 		(start 144.9125 79.405)
 		(end 143.78 80.5375)
-		(width 0.25)
+		(width 0.5)
 		(layer "F.Cu")
 		(net 3)
@@
 		(start 143.78 80.5375)
 		(end 143.78 83.21)
-		(width 0.25)
+		(width 0.5)
 		(layer "F.Cu")
 		(net 3)
@@
 		(start 134.9375 88.225)
 		(end 135.5 88.7875)
-		(width 0.5)
+		(width 0.65)
 		(layer "F.Cu")
 		(net 4)
@@
 		(start 131.29 88.805)
 		(end 135.4825 88.805)
-		(width 0.5)
+		(width 0.65)
 		(layer "F.Cu")
 		(net 4)
@@
 		(start 139.385 76.865)
 		(end 134.9375 81.3125)
-		(width 0.5)
+		(width 0.65)
 		(layer "F.Cu")
 		(net 4)
@@
 		(start 144.9125 76.865)
 		(end 139.385 76.865)
-		(width 0.5)
+		(width 0.65)
 		(layer "F.Cu")
 		(net 4)
@@
 		(start 134.9375 81.3125)
 		(end 134.9375 88.225)
-		(width 0.5)
+		(width 0.65)
 		(layer "F.Cu")
 		(net 4)

Commit message: Add files via upload
Parts:
- J2: value Display OLED -> OLED
- moved J2 1.30 mm to (129.0, 74.2)
Routing:
- net Net-(D1-A): track 69.7 -> 68.9 mm
- net GND: vias 3 -> 20
Other:
- board text added: "+12VDC"
- board text added: "RESET"

Commit message: Add files via upload
Parts:
- Q1: value IRF3205N -> IRLZ44N
Changed lines of the file:
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@@
 	(title_block
 		(title "ReFlow PCB with ATtiny85-20S_50 x 70")
-		(date "2026-03-05")
+		(date "2026-03-12")
 		(rev "V2.1")
 		(company "Z32IT")
@@
 		(tags "Through hole pin header THT 2x03 2.54mm double row")
 		(property "Reference" "J3"
-			(at 1.275 -2.475 180)
+			(at 1.275 -2.475 0)
 			(layer "F.SilkS")
 			(effects
@@
 		)
 		(property "Datasheet" "~"
-			(at 0 0 270)
+			(at 0 0 90)
 			(layer "F.Fab")
 			(hide yes)
@@
 			)
 		)
-		(property "Description" ""
-			(at 0 0 270)
+		(property "Description" "Prog. interface"
+			(at 0 0 90)
 			(layer "F.Fab")
 			(hide yes)
@@
 		(sheetname "/")
 		(sheetfile "50x70_tiny.kicad_sch")
-		(attr through_hole)
+		(attr through_hole exclude_from_bom)
 		(fp_line
 			(start -1.33 6.41)
@@
 			)
 		)
-		(property "Value" "IRF3205N"
+		(property "Value" "IRLZ44N"
 			(at 2.54 2.5 180)
 			(layer "F.Fab")
@@
 		(start 139.385 76.865)
 		(end 134.9375 81.3125)
-		(width 0.35)
+		(width 0.5)
 		(layer "F.Cu")
 		(net 4)
@@
 		(start 144.9125 76.865)
 		(end 139.385 76.865)
-		(width 0.35)
+		(width 0.5)
 		(layer "F.Cu")
 		(net 4)
@@
 		(start 134.9375 81.3125)
 		(end 134.9375 88.225)
-		(width 0.35)
+		(width 0.5)
 		(layer "F.Cu")
 		(net 4)

Commit message: Add files via upload
Parts:
- removed the U2 at (141.5, 88.2)
- added R10: 10K, Resistor_SMD:R_0805_2012Metric, F.Cu at (133.0, 78.8)
- added R9: 10K, Resistor_SMD:R_0805_2012Metric, F.Cu at (133.0, 74.5)
- added U1: L7805, Package_TO_SOT_SMD:TO-252-2, F.Cu at (141.2, 88.4)
- C1: value 330n -> 1u
- C2: value 10n -> 100n
- J2: value OLED -> Display OLED
- J3: value Conn_02x03_M -> Prog.interface
- moved D1 3.17 mm to (124.2, 80.3)
- moved R5 3.17 mm to (124.2, 75.6)
- moved C1 0.90 mm to (135.5, 83.8), turned to 90 degrees
- renumbered U3 to U2
Routing:
- net +5V: track 109.2 -> 114.0 mm
- net Net-(D1-A): track 68.9 -> 73.3 mm, vias 0 -> 4
- net VCC: track 2099.2 -> 2101.0 mm, vias 2 -> 0
- net Net-(J2-Pin_2): vias 2 -> 0
- net GND: vias 20 -> 25

Commit message: Add files via upload
Parts:
- removed R10, R9: 10K, Resistor_SMD:R_0805_2012Metric
- added JP1: ~, Connector_PinHeader_2.54mm:PinHeader_1x02_P2.54mm_Vertical, F.Cu at (135.5, 85.2)
- J1: value Barrel_Jack_MountingPin -> Screw_Terminal_01x02; footprint Connector_BarrelJack:BarrelJack_Horizontal -> TerminalBlock_Phoenix:TerminalBlock_Phoenix_MKDS-1,5-2-5.08_1x02_P5.08mm_Horizontal
- SW1: value SW_MEC_5E -> ENTER; footprint Button_Switch_THT:SW_PUSH_6mm_H4.3mm -> Button_Switch_THT:SW_PUSH_6mm_H9.5mm
- SW2: value SW_MEC_5E -> SELECT; footprint Button_Switch_THT:SW_PUSH_6mm_H4.3mm -> Button_Switch_THT:SW_PUSH_6mm_H9.5mm
- SW3: value SW_MEC_5E -> RESET; footprint Button_Switch_THT:SW_PUSH_6mm_H4.3mm -> Button_Switch_THT:SW_PUSH_6mm_H9.5mm
- moved C1 10.9 mm to (146.0, 86.8), turned to -90 degrees
- moved J1 9.35 mm to (119.3, 75.3), turned to 180 degrees
- moved C3 1.12 mm to (114.0, 87.8)
- moved C2 1.00 mm to (148.0, 82.2)
Connections:
- J1 pad 1: VCC -> GND
- J1 pad 2: GND -> VCC
- Q1 pad 1: Net-(D1-A) -> Net-(JP1-B)
- R1 pad 1: Net-(D1-A) -> Net-(JP1-B)
Routing:
- net VCC: track 2101.0 -> 2118.5 mm, vias 0 -> 2
- net Net-(JP1-B): track 0.00 -> 8.52 mm
- net Net-(D1-A): track 73.3 -> 66.5 mm, vias 4 -> 2
- net +5V: track 114.0 -> 108.0 mm, vias 2 -> 0
- net GND: vias 25 -> 42
Other:
- board text added: "+12VDC/10A"
- board text added: "+5V"
- board text added: "GND"
- board text added: "MISO"
- board text added: "MOSI"
- board text added: "RST"
- board text added: "ReFlow"
- board text added: "SCK"
- board text added: "Z32IT"
- board text removed: "+12VDC"
