File: ReFlow PCB.kicad_sch (KiCad schematic)
At the start: 22 parts, among them J1 Barrel_Jack_MountingPin, J2 Display OLED, J3 Conn_02x03_M, Q1 IRF3205N, SW1 SW_MEC_5E, SW2 SW_MEC_5E, SW3 SW_MEC_5E, U2 L7805, U3 ATtiny85-20S

Commit message: Add files via upload
Parts:
- J3: value Conn_02x03_M -> Prog.interface
- Q1: value IRF3205N -> IRLZ44N
Connections:
- net at SW3.1: now also J3.6 (Pin_6), R8.1, U3.1 (~{RESET}/PB5)
Changed lines of the file:
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@@
 	(title_block
 		(title "ReFlow PCB with ATtiny85-20S_50 x 70")
-		(date "2026-02-17")
-		(rev "V2.0")
+		(date "2026-03-12")
+		(rev "V2.1")
 		(company "Z32IT")
 	)
+	(text_box "1=+5Vcc_pin8, 2=PB1_pin6, 3=PB0_pin5, 4=PB2_pin7, 5=GND_pin4, 6=PB5_pin1\n/MOSI-MISO-CLK-RST"
+		(exclude_from_sim no)
+		(at 203.2 88.9 0)
+		(size 25.4 8.89)
+		(margins 0.9525 0.9525 0.9525 0.9525)
+		(stroke
+			(width 0)
+			(type solid)
+		)
+		(fill
+			(type none)
+		)
+		(effects
+			(font
+				(size 1 1)
+			)
+			(justify left top)
+		)
+	)
 	(junction
 		(at 153.67 125.73)
@@
 			)
 		)
-		(property "Value" "Conn_02x03_M"
+		(property "Value" "Prog.interface"
 			(at 185.42 85.09 0)
 			(effects
@@
 		(on_board yes)
 		(dnp no)
-		(fields_autoplaced yes)
 		(property "Reference" "Q1"
-			(at 168.91 78.7399 0)
+			(at 168.148 80.01 0)
 			(effects
 				(font
@@
 			)
 		)
-		(property "Value" "IRF3205N"
-			(at 168.91 81.2799 0)
+		(property "Value" "IRLZ44N"
+			(at 156.464 74.422 0)
 			(effects
 				(font
@@
 			)
 		)
-		(property "Description" ""
+		(property "Description" "3950"
 			(at 134.62 104.14 0)
 			(effects

Commit message: Add files via upload
Parts:
- removed U2: L7805, Package_TO_SOT_SMD:TO-252-2, symbol Regulator_Linear:L78L05_TO92
- added R10, R9: 10K, Resistor_SMD:R_0805_2012Metric, symbol Device:R_Small
- added U1: L7805, Package_TO_SOT_SMD:TO-252-2, symbol Regulator_Linear:L7805
- C1: value 330n -> 1u
- C2: value 10n -> 100n
- renumbered U3 to U2
Connections:
- net +5V: now also R10.1, R9.1, U1.3 (OUT)
- net GND: now also U1.2 (GND)
- net VCC: now also U1.1 (IN)
- net at SW3.1: now also J3.6 (Pin_6), R8.1, U2.1 (~{RESET}/PB5)
- net at J2.1 (Pin_1), J3.3 (Pin_3), U2.5 (AREF/PB0): now also R9.2
- net at J2.2 (Pin_2), J3.4 (Pin_4), U2.7 (PB2): now also R10.2

Commit message: Add files via upload
Parts:
- removed J1: Barrel_Jack_MountingPin, Connector_BarrelJack:BarrelJack_Horizontal, symbol Connector:Barrel_Jack_MountingPin
- removed R10, R9: 10K, Resistor_SMD:R_0805_2012Metric, symbol Device:R_Small
- added J1: Screw_Terminal_01x02, TerminalBlock_Phoenix:TerminalBlock_Phoenix_MKDS-1,5-2-5.08_1x02_P5.08mm_Horizontal, symbol Connector:Screw_Terminal_01x02
- added JP1: (no value), Connector_PinHeader_2.54mm:PinHeader_1x02_P2.54mm_Vertical, symbol Jumper:Jumper_2_Small_Open
- SW1: value SW_MEC_5E -> ENTER; footprint Button_Switch_THT:SW_PUSH_6mm_H4.3mm -> Button_Switch_THT:SW_PUSH_6mm_H9.5mm
- SW2: value SW_MEC_5E -> SELECT; footprint Button_Switch_THT:SW_PUSH_6mm_H4.3mm -> Button_Switch_THT:SW_PUSH_6mm_H9.5mm
- SW3: value SW_MEC_5E -> RESET; footprint Button_Switch_THT:SW_PUSH_6mm_H4.3mm -> Button_Switch_THT:SW_PUSH_6mm_H9.5mm
Connections:
- net GND: now also J1.1 (Pin_1)
- net VCC: now also J1.2 (Pin_2)
- net at D1.2 (A), J3.2 (Pin_2), U2.6 (PB1): now also JP1.1 (A); no longer Q1.1 (G), R1.1
- net at SW3.1: now also J3.6 (Pin_6), R8.1, U2.1 (~{RESET}/PB5)
- new net: JP1.2 (B), Q1.1 (G), R1.1
Other:
- note added: "Input voltage 12V/10A"
- note added: "JP1 Open-Prog.mode/Closed-normal mode"
- moved on the sheet: C1, C2, C3, D1, R1, R5, U1
